File: Kicad_Controller/Nintendo_wireless_controller_curcuit.sch (KiCad schematic (older format))
At the start: 13 parts, among them IC1 ATTINY2313-S, J1 NRF_conn, J2 BATT, X1 8MHz, X1 USB-MB-S

Commit message: added approximated power consumption, started pcb layout, finished some of wireless module schematic
Parts:
- added C? (x2): 1uF, symbol CP1
- added C?: 100n, symbol C
- added C?: 10u, symbol CP1
- added U?: LP5951MF-3.3, MODULE, symbol LP5951MF-3.3
- added sw1: CONN_2, symbol CONN_2
Connections:
- net +BATT: now also sw1.2 (PM)
- net GND: now also IC1.10 (GND), J1.1, C?.2, C?.2, C?.2, C?.2, U?.2 (GND)
- net VCC: now also IC1.20 (VCC), J1.2, C?.1, C?.1, C?.1, U?.5 (Vout)
- net CE: now reaches J1.3
- net CE: now also IC1.15 ((PCINT3/OC1A)PB3)
- net CSN: now reaches J1.4
- net CSN: now also IC1.16 ((PCINT4/OC1B)PB4)
- net SCK: now reaches J1.5
- net SCK: now also IC1.19 ((PCINT7/USCK/SCK/SCL)PB7)
- net MOSI: now reaches J1.6
- net MOSI: now also IC1.17 ((PCINT5/MOSI/DI/SDA)PB5)
- net MISO: now reaches J1.7
- net MISO: now also IC1.18 ((PCINT6/MISO/DO)PB6)
- net IRQ: now reaches J1.8
- net IRQ: now also IC1.14 ((PCINT2/OC0A)PB2)
- new net: C?.1, U?.1 (Vin), U?.3 (Ven), sw1.1 (P1)
Other:
- note added: "2mA Avg."
- note added: "3mA@3v3@8MHz"
- note added: "70uA@150mA load"

Commit message: board layout done for Kicad_N64
Parts:
- gave numbers to parts that had none: 13
- renumbered J2 to J1, J1 to J2, X1 to X2
Connections:
- net VCC: now also R2.2
- no-connect marks 0 -> 12
