File: Basestation_Hardware_Kicad/$N64_USB_FTW.sch (KiCad schematic (older format))
At the start: 28 parts, among them IC1 ATMEGA8-AI, U1 LM317, X1 12mhz, X2 USB

Commit message: fiddle diddle
Parts:
- renumbered GC to GC1, NRF to NRF1, PROG to PROG1
Changed lines of the file:
@@
-EESchema Schematic File Version 2  date 19-06-2012 12:50:49
+EESchema Schematic File Version 2  date 19-06-2012 13:01:28
 LIBS:power
 LIBS:device
@@
 MCU_VCC
 $Comp
-L CONN_5X2 NRF
+L CONN_5X2 NRF1
 U 1 1 4F68E2A7
 P 6950 6750
-F 0 "NRF" H 6950 7050 60  0000 C CNN
+F 0 "NRF1" H 6950 7050 60  0000 C CNN
 F 1 "CONN_5X2" V 6950 6750 50  0000 C CNN
 	1    6950 6750
@@
 $EndComp
 $Comp
-L GND #PWR01
+L GND #PWR17
 U 1 1 4F56953B
 P 12000 2950
-F 0 "#PWR01" H 12000 2950 30  0001 C CNN
+F 0 "#PWR17" H 12000 2950 30  0001 C CNN
 F 1 "GND" H 12000 2880 30  0001 C CNN
 	1    12000 2950
@@
 $EndComp
 $Comp
-L GND #PWR02
+L GND #PWR15
 U 1 1 4F56949A
 P 10600 3050
-F 0 "#PWR02" H 10600 3050 30  0001 C CNN
+F 0 "#PWR15" H 10600 3050 30  0001 C CNN
 F 1 "GND" H 10600 2980 30  0001 C CNN
 	1    10600 3050
@@
 $EndComp
 $Comp
-L GND #PWR03
+L GND #PWR7
 U 1 1 4F5646E2
 P 4450 4700
-F 0 "#PWR03" H 4450 4700 30  0001 C CNN
+F 0 "#PWR7" H 4450 4700 30  0001 C CNN
 F 1 "GND" H 4450 4630 30  0001 C CNN
 	1    4450 4700
@@
 $EndComp
 $Comp
-L GND #PWR04
+L GND #PWR4
 U 1 1 4F563B84
 P 3600 5700
-F 0 "#PWR04" H 3600 5700 30  0001 C CNN
+F 0 "#PWR4" H 3600 5700 30  0001 C CNN
 F 1 "GND" H 3600 5630 30  0001 C CNN
 	1    3600 5700
@@
 $EndComp
 $Comp
-L VCC #PWR05
+L VCC #PWR12
 U 1 1 4F563AF3
 P 9350 2200
-F 0 "#PWR05" H 9350 2300 30  0001 C CNN
+F 0 "#PWR12" H 9350 2300 30  0001 C CNN
 F 1 "VCC" H 9350 2300 30  0000 C CNN
 	1    9350 2200
@@
 MCU_VCC
 $Comp
-L GND #PWR06
+L GND #PWR1
 U 1 1 4F4E474C
 P 1800 4050
-F 0 "#PWR06" H 1800 4050 30  0001 C CNN
+F 0 "#PWR1" H 1800 4050 30  0001 C CNN
 F 1 "GND" H 1800 3980 30  0001 C CNN
 	1    1800 4050
@@
 $EndComp
 $Comp
-L GND #PWR07
+L GND #PWR3
 U 1 1 4F4D32A1
 P 3150 5700
-F 0 "#PWR07" H 3150 5700 30  0001 C CNN
+F 0 "#PWR3" H 3150 5700 30  0001 C CNN
 F 1 "GND" H 3150 5630 30  0001 C CNN
 	1    3150 5700
@@
 SCK
 $Comp
-L GND #PWR08
+L GND #PWR8
 U 1 1 4F4D25F3
 P 6300 7100
-F 0 "#PWR08" H 6300 7100 30  0001 C CNN
+F 0 "#PWR8" H 6300 7100 30  0001 C CNN
 F 1 "GND" H 6300 7030 30  0001 C CNN
 	1    6300 7100
@@
 $EndComp
 $Comp
-L GND #PWR09
+L GND #PWR19
 U 1 1 4F4D1C43
 P 12300 4050
-F 0 "#PWR09" H 12300 4050 30  0001 C CNN
+F 0 "#PWR19" H 12300 4050 30  0001 C CNN
 F 1 "GND" H 12300 3980 30  0001 C CNN
 	1    12300 4050
@@
 $EndComp
 $Comp
-L GND #PWR010
+L GND #PWR18
 U 1 1 4F452EB3
 P 12200 6250
-F 0 "#PWR010" H 12200 6250 30  0001 C CNN
+F 0 "#PWR18" H 12200 6250 30  0001 C CNN
 F 1 "GND" H 12200 6180 30  0001 C CNN
 	1    12200 6250
@@
 Controller Data
 $Comp
-L VCC #PWR011
+L VCC #PWR16
 U 1 1 4F452CF5
 P 11950 5000
-F 0 "#PWR011" H 11950 5100 30  0001 C CNN
+F 0 "#PWR16" H 11950 5100 30  0001 C CNN
 F 1 "VCC" H 11950 5100 30  0000 C CNN
 	1    11950 5000
@@
 GC_Controller
 $Comp
-L CONN_7 GC
+L CONN_7 GC1
 U 1 1 4F452C08
 P 11200 5500
-F 0 "GC" V 11170 5500 60  0000 C CNN
+F 0 "GC1" V 11170 5500 60  0000 C CNN
 F 1 "CONN_7" V 11270 5500 60  0000 C CNN
 	1    11200 5500
@@
 $EndComp
 $Comp
-L GND #PWR012
+L GND #PWR20
 U 1 1 4F45295F
 P 12850 3050
-F 0 "#PWR012" H 12850 3050 30  0001 C CNN
+F 0 "#PWR20" H 12850 3050 30  0001 C CNN
 F 1 "GND" H 12850 2980 30  0001 C CNN
 	1    12850 3050
@@
 $EndComp
 $Comp
-L GND #PWR013
+L GND #PWR14
 U 1 1 4F45213D
 P 9900 2950
-F 0 "#PWR013" H 9900 2950 30  0001 C CNN
+F 0 "#PWR14" H 9900 2950 30  0001 C CNN
 F 1 "GND" H 9900 2880 30  0001 C CNN
 	1    9900 2950
@@
 $EndComp
 $Comp
-L GND #PWR014
+L GND #PWR11
 U 1 1 4F440011
 P 9100 3850
-F 0 "#PWR014" H 9100 3850 30  0001 C CNN
+F 0 "#PWR11" H 9100 3850 30  0001 C CNN
 F 1 "GND" H 9100 3780 30  0001 C CNN
 	1    9100 3850
@@
 pc5
 $Comp
-L GND #PWR015
+L GND #PWR9
 U 1 1 4F43FD84
 P 6750 2200
-F 0 "#PWR015" H 6750 2200 30  0001 C CNN
+F 0 "#PWR9" H 6750 2200 30  0001 C CNN
 F 1 "GND" H 6750 2130 30  0001 C CNN
 	1    6750 2200
@@
 $EndComp
 $Comp
-L GND #PWR016
+L GND #PWR10
 U 1 1 4F43FD6B
 P 6850 2200
-F 0 "#PWR016" H 6850 2200 30  0001 C CNN
+F 0 "#PWR10" H 6850 2200 30  0001 C CNN
 F 1 "GND" H 6850 2130 30  0001 C CNN
 	1    6850 2200
@@
 $EndComp
 $Comp
-L GND #PWR017
+L GND #PWR13
 U 1 1 4F43FC5C
 P 9500 5000
-F 0 "#PWR017" H 9500 5000 30  0001 C CNN
+F 0 "#PWR13" H 9500 5000 30  0001 C CNN
 F 1 "GND" H 9500 4930 30  0001 C CNN
 	1    9500 5000
@@
 SCK
 $Comp
-L GND #PWR018
+L GND #PWR2
 U 1 1 4F43F2E9
 P 3100 4750
-F 0 "#PWR018" H 3100 4750 30  0001 C CNN
+F 0 "#PWR2" H 3100 4750 30  0001 C CNN
 F 1 "GND" H 3100 4680 30  0001 C CNN
 	1    3100 4750
@@
 $EndComp
 $Comp
-L GND #PWR019
+L GND #PWR6
 U 1 1 4F43EE47
 P 3800 4750
-F 0 "#PWR019" H 3800 4750 30  0001 C CNN
+F 0 "#PWR6" H 3800 4750 30  0001 C CNN
 F 1 "GND" H 3800 4680 30  0001 C CNN
 	1    3800 4750
@@
 $EndComp
 $Comp
-L CONN_3X2 PROG
+L CONN_3X2 PROG1
 U 1 1 4F43E0D8
 P 9100 4750
-F 0 "PROG" H 9100 5000 50  0000 C CNN
+F 0 "PROG1" H 9100 5000 50  0000 C CNN
 F 1 "CONN_3X2" V 9100 4800 40  0000 C CNN
 	1    9100 4750
@@
 $EndComp
 $Comp
-L VCC #PWR020
+L VCC #PWR5
 U 1 1 4F43DEFD
 P 3650 2900
-F 0 "#PWR020" H 3650 3000 30  0001 C CNN
+F 0 "#PWR5" H 3650 3000 30  0001 C CNN
 F 1 "VCC" H 3650 3000 30  0000 C CNN
 	1    3650 2900
