File: Controller_Hardware_Kicad/Nintendo_wireless_controller_curcuit.sch (KiCad schematic (older format))
At the start: 19 parts, among them IC1 ATTINY2313-S, J1 BATT, J2 NRF_conn, U1 MAX1811, U2 LP5951MF-3.3, X1 USB-MB-S, X2 8MHz, sw1 CONN_2

Commit message: Finished routing the controller
Parts:
- added C10, C9: 100n, symbol C
- added Center_VCC1, Side_VCC1: CONN_2, symbol CONN_2
- C7: value 1uF -> 4.7uF
- R2: value R -> 100K
Connections:
- net +5V: now also C10.1
- net GND: now also C10.2, C9.2, Side_VCC1.1 (P1); no longer C1.1, C2.1, C3.2, C4.2, IC1.10 (GND), J2.1
- net VCC: now also Side_VCC1.2 (PM); no longer C3.1, C4.1, IC1.20 (VCC), J2.2, R2.2
- net at C7.1, U2.1 (Vin), U2.3 (Ven)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: now also C9.1
- new net +3.3V: C3.1, C4.1, Center_VCC1.1 (P1), IC1.20 (VCC), J2.2, R2.2
- new net DGND: C1.1, C2.1, C3.2, C4.2, Center_VCC1.2 (PM), IC1.10 (GND), J2.1
Other:
- moved on the sheet: C1, C2, C3, C4, C7, C8, IC1, J2, R2, U2, X2, sw1

Commit message: continued Part sourcing - added some missing values to both designs
Parts:
- C1, C2: value C -> 27p
Changed lines of the file:
@@
-EESchema Schematic File Version 2  date 31-05-2012 10:27:24
+EESchema Schematic File Version 2  date 04-06-2012 17:42:45
 LIBS:power
 LIBS:device
@@
 Sheet 1 1
 Title ""
-Date "31 may 2012"
+Date "4 jun 2012"
 Rev ""
 Comp ""
@@
 $EndComp
 $Comp
-L +3.3V #PWR24
+L +3.3V #PWR01
 U 1 1 4FC72ABF
 P 8300 2300
-F 0 "#PWR24" H 8300 2260 30  0001 C CNN
+F 0 "#PWR01" H 8300 2260 30  0001 C CNN
 F 1 "+3.3V" H 8300 2410 30  0000 C CNN
 	1    8300 2300
@@
 $EndComp
 $Comp
-L +3.3V #PWR11
+L +3.3V #PWR02
 U 1 1 4FC72ABB
 P 4450 1250
-F 0 "#PWR11" H 4450 1210 30  0001 C CNN
+F 0 "#PWR02" H 4450 1210 30  0001 C CNN
 F 1 "+3.3V" H 4450 1360 30  0000 C CNN
 	1    4450 1250
@@
 $EndComp
 $Comp
-L +3.3V #PWR8
+L +3.3V #PWR03
 U 1 1 4FC72AB8
 P 3300 700
-F 0 "#PWR8" H 3300 660 30  0001 C CNN
+F 0 "#PWR03" H 3300 660 30  0001 C CNN
 F 1 "+3.3V" H 3300 810 30  0000 C CNN
 	1    3300 700
@@
 $EndComp
 $Comp
-L +3.3V #PWR6
+L +3.3V #PWR04
 U 1 1 4FC72AB1
 P 2600 2950
-F 0 "#PWR6" H 2600 2910 30  0001 C CNN
+F 0 "#PWR04" H 2600 2910 30  0001 C CNN
 F 1 "+3.3V" H 2600 3060 30  0000 C CNN
 	1    2600 2950
@@
 $EndComp
 $Comp
-L +3.3V #PWR15
+L +3.3V #PWR05
 U 1 1 4FC72AA1
 P 5150 4150
-F 0 "#PWR15" H 5150 4110 30  0001 C CNN
+F 0 "#PWR05" H 5150 4110 30  0001 C CNN
 F 1 "+3.3V" H 5150 4260 30  0000 C CNN
 	1    5150 4150
@@
 $EndComp
 $Comp
-L VCC #PWR17
+L VCC #PWR06
 U 1 1 4FC72A8E
 P 5650 4950
-F 0 "#PWR17" H 5650 5050 30  0001 C CNN
+F 0 "#PWR06" H 5650 5050 30  0001 C CNN
 F 1 "VCC" H 5650 5050 30  0000 C CNN
 	1    5650 4950
@@
 $EndComp
 $Comp
-L GND #PWR18
+L GND #PWR07
 U 1 1 4FC72A57
 P 5650 5300
-F 0 "#PWR18" H 5650 5300 30  0001 C CNN
+F 0 "#PWR07" H 5650 5300 30  0001 C CNN
 F 1 "GND" H 5650 5230 30  0001 C CNN
 	1    5650 5300
@@
 $EndComp
 $Comp
-L DGND #PWR21
+L DGND #PWR08
 U 1 1 4FC72A50
 P 6750 2700
-F 0 "#PWR21" H 6750 2700 40  0001 C CNN
+F 0 "#PWR08" H 6750 2700 40  0001 C CNN
 F 1 "DGND" H 6750 2630 40  0000 C CNN
 	1    6750 2700
@@
 $EndComp
 $Comp
-L DGND #PWR2
+L DGND #PWR09
 U 1 1 4FC72A1D
 P 1750 2700
-F 0 "#PWR2" H 1750 2700 40  0001 C CNN
+F 0 "#PWR09" H 1750 2700 40  0001 C CNN
 F 1 "DGND" H 1750 2630 40  0000 C CNN
 	1    1750 2700
@@
 $EndComp
 $Comp
-L DGND #PWR7
+L DGND #PWR010
 U 1 1 4FC72A04
 P 2600 3650
-F 0 "#PWR7" H 2600 3650 40  0001 C CNN
+F 0 "#PWR010" H 2600 3650 40  0001 C CNN
 F 1 "DGND" H 2600 3580 40  0000 C CNN
 	1    2600 3650
@@
 $EndComp
 $Comp
-L DGND #PWR12
+L DGND #PWR011
 U 1 1 4FC729FC
 P 4450 3600
-F 0 "#PWR12" H 4450 3600 40  0001 C CNN
+F 0 "#PWR011" H 4450 3600 40  0001 C CNN
 F 1 "DGND" H 4450 3530 40  0000 C CNN
 	1    4450 3600
@@
 $EndComp
 $Comp
-L DGND #PWR16
+L DGND #PWR012
 U 1 1 4FC729EC
 P 5150 4500
-F 0 "#PWR16" H 5150 4500 40  0001 C CNN
+F 0 "#PWR012" H 5150 4500 40  0001 C CNN
 F 1 "DGND" H 5150 4430 40  0000 C CNN
 	1    5150 4500
@@
 $EndComp
 $Comp
-L GND #PWR23
+L GND #PWR013
 U 1 1 4F5F6BBA
 P 7550 6550
-F 0 "#PWR23" H 7550 6550 30  0001 C CNN
+F 0 "#PWR013" H 7550 6550 30  0001 C CNN
 F 1 "GND" H 7550 6480 30  0001 C CNN
 	1    7550 6550
@@
 $EndComp
 $Comp
-L GND #PWR27
+L GND #PWR014
 U 1 1 4F5F6A53
 P 10150 6500
-F 0 "#PWR27" H 10150 6500 30  0001 C CNN
+F 0 "#PWR014" H 10150 6500 30  0001 C CNN
 F 1 "GND" H 10150 6430 30  0001 C CNN
 	1    10150 6500
@@
 $EndComp
 $Comp
-L GND #PWR25
+L GND #PWR015
 U 1 1 4F5F6856
 P 8900 6850
-F 0 "#PWR25" H 8900 6850 30  0001 C CNN
+F 0 "#PWR015" H 8900 6850 30  0001 C CNN
 F 1 "GND" H 8900 6780 30  0001 C CNN
 	1    8900 6850
@@
 $EndComp
 $Comp
-L +5V #PWR4
+L +5V #PWR016
 U 1 1 4F4F395E
 P 2150 5300
-F 0 "#PWR4" H 2150 5390 20  0001 C CNN
+F 0 "#PWR016" H 2150 5390 20  0001 C CNN
 F 1 "+5V" H 2150 5390 30  0000 C CNN
 	1    2150 5300
@@
 $EndComp
 $Comp
-L +5V #PWR13
+L +5V #PWR017
 U 1 1 4F4F393F
 P 4450 6600
-F 0 "#PWR13" H 4450 6690 20  0001 C CNN
+F 0 "#PWR017" H 4450 6690 20  0001 C CNN
 F 1 "+5V" H 4450 6690 30  0000 C CNN
 	1    4450 6600
@@
 $EndComp
 $Comp
-L GND #PWR14
+L GND #PWR018
 U 1 1 4F4F3934
 P 4450 7300
-F 0 "#PWR14" H 4450 7300 30  0001 C CNN
+F 0 "#PWR018" H 4450 7300 30  0001 C CNN
 F 1 "GND" H 4450 7230 30  0001 C CNN
 	1    4450 7300
@@
 $EndComp
 $Comp
-L +BATT #PWR9
+L +BATT #PWR019
 U 1 1 4F4F390D
 P 4000 6350
-F 0 "#PWR9" H 4000 6300 20  0001 C CNN
+F 0 "#PWR019" H 4000 6300 20  0001 C CNN
 F 1 "+BATT" H 4000 6450 30  0000 C CNN
 	1    4000 6350
@@
 $EndComp
 $Comp
-L GND #PWR10
+L GND #PWR020
 U 1 1 4F4F38CA
 P 4000 7100
-F 0 "#PWR10" H 4000 7100 30  0001 C CNN
+F 0 "#PWR020" H 4000 7100 30  0001 C CNN
 F 1 "GND" H 4000 7030 30  0001 C CNN
 	1    4000 7100
@@
 $EndComp
 $Comp
-L GND #PWR5
+L GND #PWR021
 U 1 1 4F4F38C1
 P 2550 7100
-F 0 "#PWR5" H 2550 7100 30  0001 C CNN
+F 0 "#PWR021" H 2550 7100 30  0001 C CNN
 F 1 "GND" H 2550 7030 30  0001 C CNN
 	1    2550 7100
@@
 $EndComp
 $Comp
-L GND #PWR20
+L GND #PWR022
 U 1 1 4F4F372C
 P 5700 7150
-F 0 "#PWR20" H 5700 7150 30  0001 C CNN
+F 0 "#PWR022" H 5700 7150 30  0001 C CNN
 F 1 "GND" H 5700 7080 30  0001 C CNN
 	1    5700 7150
@@
 $EndComp
 $Comp
-L +BATT #PWR19
+L +BATT #PWR023
 U 1 1 4F4F3725
 P 5700 6500
-F 0 "#PWR19" H 5700 6450 20  0001 C CNN
+F 0 "#PWR023" H 5700 6450 20  0001 C CNN
 F 1 "+BATT" H 5700 6600 30  0000 C CNN
 	1    5700 6500
@@
 $EndComp
 $Comp
-L +BATT #PWR22
+L +BATT #PWR024
 U 1 1 4F4F36FD
 P 7550 5400
-F 0 "#PWR22" H 7550 5350 20  0001 C CNN
+F 0 "#PWR024" H 7550 5350 20  0001 C CNN
 F 1 "+BATT" H 7550 5500 30  0000 C CNN
 	1    7550 5400
@@
 $EndComp
 $Comp
-L VCC #PWR26
+L VCC #PWR025
 U 1 1 4F4F36D4
 P 9750 5550
-F 0 "#PWR26" H 9750 5650 30  0001 C CNN
+F 0 "#PWR025" H 9750 5650 30  0001 C CNN
 F 1 "VCC" H 9750 5650 30  0000 C CNN
 	1    9750 5550
@@
 $EndComp
 $Comp
-L GND #PWR1
+L GND #PWR026
 U 1 1 4F4F36B2
 P 1500 5700
-F 0 "#PWR1" H 1500 5700 30  0001 C CNN
+F 0 "#PWR026" H 1500 5700 30  0001 C CNN
 F 1 "GND" H 1500 5630 30  0001 C CNN
 	1    1500 5700
@@
 $EndComp
 $Comp
-L +5V #PWR3
+L +5V #PWR027
 U 1 1 4F4F36A7
 P 1750 5300
-F 0 "#PWR3" H 1750 5390 20  0001 C CNN
+F 0 "#PWR027" H 1750 5390 20  0001 C CNN
 F 1 "+5V" H 1750 5390 30  0000 C CNN
 	1    1750 5300
@@
 P 2100 2550
 F 0 "C2" H 2150 2650 50  0000 L CNN
-F 1 "C" H 2150 2450 50  0000 L CNN
+F 1 "27p" H 2150 2450 50  0000 L CNN
 	1    2100 2550
 	0    -1   -1   0
@@
 P 2100 1750
 F 0 "C1" H 2150 1850 50  0000 L CNN
-F 1 "C" H 2150 1650 50  0000 L CNN
+F 1 "27p" H 2150 1650 50  0000 L CNN
 	1    2100 1750
 	0    -1   -1   0

Commit message: load caps on xtals changed from 27pf to 22pf
Parts:
- C1, C2: value 27p -> 22pf
Changed lines of the file:
@@
-EESchema Schematic File Version 2  date 04-06-2012 17:42:45
+EESchema Schematic File Version 2  date 19-06-2012 13:27:23
 LIBS:power
 LIBS:device
@@
 Sheet 1 1
 Title ""
-Date "4 jun 2012"
+Date "19 jun 2012"
 Rev ""
 Comp ""
@@
 P 2100 2550
 F 0 "C2" H 2150 2650 50  0000 L CNN
-F 1 "27p" H 2150 2450 50  0000 L CNN
+F 1 "22pf" H 2150 2450 50  0000 L CNN
 	1    2100 2550
 	0    -1   -1   0
@@
 P 2100 1750
 F 0 "C1" H 2150 1850 50  0000 L CNN
-F 1 "27p" H 2150 1650 50  0000 L CNN
+F 1 "22pf" H 2150 1650 50  0000 L CNN
 	1    2100 1750
 	0    -1   -1   0

Commit message: configured max1811 pin connections to correct settings
Connections:
- net +5V: now also U1.1 (SELV)
- net GND: no longer U1.1 (SELV)
Other:
- note added: "100mA charge current = ca. 4hr charge time"
Changed lines of the file:
@@
-EESchema Schematic File Version 2  date 19-06-2012 13:27:23
+EESchema Schematic File Version 2  date 19-06-2012 16:34:13
 LIBS:power
 LIBS:device
@@
 Comment4 ""
 $EndDescr
+Text Notes 2850 6150 0    60   ~ 0
+100mA charge current = ca. 4hr charge time
+Wire Wire Line
+	2550 7100 2550 6800
 Connection ~ 4450 7200
 Wire Wire Line
@@
 	2150 5350 2700 5350
 Wire Wire Line
-	2700 6500 2150 6500
-Wire Wire Line
-	2150 6500 2150 6350
+	2150 6500 2700 6500
+Wire Wire Line
+	2150 6350 2150 6500
 Wire Wire Line
 	2150 5300 2150 5400
@@
 Connection ~ 2550 6800
 Wire Wire Line
-	2700 6800 2550 6800
+	2550 6800 2700 6800
 Connection ~ 5700 7000
 Wire Wire Line
@@
 	1900 2550 1750 2550
 Wire Wire Line
-	1900 1750 1750 1750
+	1750 1750 1900 1750
 Connection ~ 1750 2550
 Wire Wire Line
@@
 	3300 2200 3200 2200
 Wire Wire Line
-	3200 2200 3200 2550
-Wire Wire Line
-	3200 2550 2300 2550
+	3200 2550 3200 2200
+Wire Wire Line
+	2300 2550 3200 2550
 Connection ~ 2400 2550
 Wire Wire Line
@@
 	2700 6700 2550 6700
 Wire Wire Line
-	2550 6700 2550 7100
-Wire Wire Line
-	2700 7000 2550 7000
+	2550 7000 2700 7000
 Connection ~ 2550 7000
 Wire Wire Line
@@
 Connection ~ 2150 6450
 Wire Wire Line
-	9700 6000 9750 6000
-Wire Wire Line
-	9750 6000 9750 5550
+	9750 6000 9700 6000
+Wire Wire Line
+	9750 5550 9750 6000
 Wire Wire Line
 	10150 6250 10150 6500
@@
 	2600 3650 2600 3550
 Wire Wire Line
-	1750 1750 1750 2700
+	1750 2700 1750 1750
 Wire Wire Line
 	5600 5200 5650 5200
@@
 Wire Wire Line
 	4800 7200 4450 7200
+Wire Wire Line
+	2550 6700 2550 6650
+$Comp
+L +5V #PWR01
+U 1 1 4FE08C10
+P 2550 6650
+F 0 "#PWR01" H 2550 6740 20  0001 C CNN
+F 1 "+5V" H 2550 6740 30  0000 C CNN
+	1    2550 6650
+	1    0    0    -1
+$EndComp
 $Comp
 L C C10
@@
 $EndComp
 $Comp
-L +3.3V #PWR01
+L +3.3V #PWR02
 U 1 1 4FC72ABF
 P 8300 2300
-F 0 "#PWR01" H 8300 2260 30  0001 C CNN
+F 0 "#PWR02" H 8300 2260 30  0001 C CNN
 F 1 "+3.3V" H 8300 2410 30  0000 C CNN
 	1    8300 2300
@@
 $EndComp
 $Comp
-L +3.3V #PWR02
+L +3.3V #PWR03
 U 1 1 4FC72ABB
 P 4450 1250
-F 0 "#PWR02" H 4450 1210 30  0001 C CNN
+F 0 "#PWR03" H 4450 1210 30  0001 C CNN
 F 1 "+3.3V" H 4450 1360 30  0000 C CNN
 	1    4450 1250
@@
 $EndComp
 $Comp
-L +3.3V #PWR03
+L +3.3V #PWR04
 U 1 1 4FC72AB8
 P 3300 700
-F 0 "#PWR03" H 3300 660 30  0001 C CNN
+F 0 "#PWR04" H 3300 660 30  0001 C CNN
 F 1 "+3.3V" H 3300 810 30  0000 C CNN
 	1    3300 700
@@
 $EndComp
 $Comp
-L +3.3V #PWR04
+L +3.3V #PWR05
 U 1 1 4FC72AB1
 P 2600 2950
-F 0 "#PWR04" H 2600 2910 30  0001 C CNN
+F 0 "#PWR05" H 2600 2910 30  0001 C CNN
 F 1 "+3.3V" H 2600 3060 30  0000 C CNN
 	1    2600 2950
@@
 $EndComp
 $Comp
-L +3.3V #PWR05
+L +3.3V #PWR06
 U 1 1 4FC72AA1
 P 5150 4150
-F 0 "#PWR05" H 5150 4110 30  0001 C CNN
+F 0 "#PWR06" H 5150 4110 30  0001 C CNN
 F 1 "+3.3V" H 5150 4260 30  0000 C CNN
 	1    5150 4150
@@
 $EndComp
 $Comp
-L VCC #PWR06
+L VCC #PWR07
 U 1 1 4FC72A8E
 P 5650 4950
-F 0 "#PWR06" H 5650 5050 30  0001 C CNN
+F 0 "#PWR07" H 5650 5050 30  0001 C CNN
 F 1 "VCC" H 5650 5050 30  0000 C CNN
 	1    5650 4950
@@
 $EndComp
 $Comp
-L GND #PWR07
+L GND #PWR08
 U 1 1 4FC72A57
 P 5650 5300
-F 0 "#PWR07" H 5650 5300 30  0001 C CNN
+F 0 "#PWR08" H 5650 5300 30  0001 C CNN
 F 1 "GND" H 5650 5230 30  0001 C CNN
 	1    5650 5300
@@
 $EndComp
 $Comp
-L DGND #PWR08
+L DGND #PWR09
 U 1 1 4FC72A50
 P 6750 2700
-F 0 "#PWR08" H 6750 2700 40  0001 C CNN
+F 0 "#PWR09" H 6750 2700 40  0001 C CNN
 F 1 "DGND" H 6750 2630 40  0000 C CNN
 	1    6750 2700
@@
 $EndComp
 $Comp
-L DGND #PWR09
+L DGND #PWR010
 U 1 1 4FC72A1D
 P 1750 2700
-F 0 "#PWR09" H 1750 2700 40  0001 C CNN
+F 0 "#PWR010" H 1750 2700 40  0001 C CNN
 F 1 "DGND" H 1750 2630 40  0000 C CNN
 	1    1750 2700
@@
 $EndComp
 $Comp
-L DGND #PWR010
+L DGND #PWR011
 U 1 1 4FC72A04
 P 2600 3650
-F 0 "#PWR010" H 2600 3650 40  0001 C CNN
+F 0 "#PWR011" H 2600 3650 40  0001 C CNN
 F 1 "DGND" H 2600 3580 40  0000 C CNN
 	1    2600 3650
@@
 $EndComp
 $Comp
-L DGND #PWR011
+L DGND #PWR012
 U 1 1 4FC729FC
 P 4450 3600
-F 0 "#PWR011" H 4450 3600 40  0001 C CNN
+F 0 "#PWR012" H 4450 3600 40  0001 C CNN
 F 1 "DGND" H 4450 3530 40  0000 C CNN
 	1    4450 3600
@@
 $EndComp
 $Comp
-L DGND #PWR012
+L DGND #PWR013
 U 1 1 4FC729EC
 P 5150 4500
-F 0 "#PWR012" H 5150 4500 40  0001 C CNN
+F 0 "#PWR013" H 5150 4500 40  0001 C CNN
 F 1 "DGND" H 5150 4430 40  0000 C CNN
 	1    5150 4500
@@
 $EndComp
 $Comp
-L GND #PWR013
+L GND #PWR014
 U 1 1 4F5F6BBA
 P 7550 6550
-F 0 "#PWR013" H 7550 6550 30  0001 C CNN
+F 0 "#PWR014" H 7550 6550 30  0001 C CNN
 F 1 "GND" H 7550 6480 30  0001 C CNN
 	1    7550 6550
@@
 $EndComp
 $Comp
-L GND #PWR014
+L GND #PWR015
 U 1 1 4F5F6A53
 P 10150 6500
-F 0 "#PWR014" H 10150 6500 30  0001 C CNN
+F 0 "#PWR015" H 10150 6500 30  0001 C CNN
 F 1 "GND" H 10150 6430 30  0001 C CNN
 	1    10150 6500
@@
 $EndComp
 $Comp
-L GND #PWR015
+L GND #PWR016
 U 1 1 4F5F6856
 P 8900 6850
-F 0 "#PWR015" H 8900 6850 30  0001 C CNN
+F 0 "#PWR016" H 8900 6850 30  0001 C CNN
 F 1 "GND" H 8900 6780 30  0001 C CNN
 	1    8900 6850
@@
 $EndComp
 $Comp
-L +5V #PWR016
+L +5V #PWR017
 U 1 1 4F4F395E
 P 2150 5300
-F 0 "#PWR016" H 2150 5390 20  0001 C CNN
+F 0 "#PWR017" H 2150 5390 20  0001 C CNN
 F 1 "+5V" H 2150 5390 30  0000 C CNN
 	1    2150 5300
@@
 $EndComp
 $Comp
-L +5V #PWR017
+L +5V #PWR018
 U 1 1 4F4F393F
 P 4450 6600
-F 0 "#PWR017" H 4450 6690 20  0001 C CNN
+F 0 "#PWR018" H 4450 6690 20  0001 C CNN
 F 1 "+5V" H 4450 6690 30  0000 C CNN
 	1    4450 6600
@@
 $EndComp
 $Comp
-L GND #PWR018
+L GND #PWR019
 U 1 1 4F4F3934
 P 4450 7300
-F 0 "#PWR018" H 4450 7300 30  0001 C CNN
+F 0 "#PWR019" H 4450 7300 30  0001 C CNN
 F 1 "GND" H 4450 7230 30  0001 C CNN
 	1    4450 7300
@@
 $EndComp
 $Comp
-L +BATT #PWR019
+L +BATT #PWR020
 U 1 1 4F4F390D
 P 4000 6350
-F 0 "#PWR019" H 4000 6300 20  0001 C CNN
+F 0 "#PWR020" H 4000 6300 20  0001 C CNN
 F 1 "+BATT" H 4000 6450 30  0000 C CNN
 	1    4000 6350
@@
 $EndComp
 $Comp
-L GND #PWR020
+L GND #PWR021
 U 1 1 4F4F38CA
 P 4000 7100
-F 0 "#PWR020" H 4000 7100 30  0001 C CNN
+F 0 "#PWR021" H 4000 7100 30  0001 C CNN
 F 1 "GND" H 4000 7030 30  0001 C CNN
 	1    4000 7100
@@
 $EndComp
 $Comp
-L GND #PWR021
+L GND #PWR022
 U 1 1 4F4F38C1
 P 2550 7100
-F 0 "#PWR021" H 2550 7100 30  0001 C CNN
+F 0 "#PWR022" H 2550 7100 30  0001 C CNN
 F 1 "GND" H 2550 7030 30  0001 C CNN
 	1    2550 7100
@@
 $EndComp
 $Comp
-L GND #PWR022
+L GND #PWR023
 U 1 1 4F4F372C
 P 5700 7150
-F 0 "#PWR022" H 5700 7150 30  0001 C CNN
+F 0 "#PWR023" H 5700 7150 30  0001 C CNN
 F 1 "GND" H 5700 7080 30  0001 C CNN
 	1    5700 7150
@@
 $EndComp
 $Comp
-L +BATT #PWR023
+L +BATT #PWR024
 U 1 1 4F4F3725
 P 5700 6500
-F 0 "#PWR023" H 5700 6450 20  0001 C CNN
+F 0 "#PWR024" H 5700 6450 20  0001 C CNN
 F 1 "+BATT" H 5700 6600 30  0000 C CNN
 	1    5700 6500
@@
 $EndComp
 $Comp
-L +BATT #PWR024
+L +BATT #PWR025
 U 1 1 4F4F36FD
 P 7550 5400
-F 0 "#PWR024" H 7550 5350 20  0001 C CNN
+F 0 "#PWR025" H 7550 5350 20  0001 C CNN
 F 1 "+BATT" H 7550 5500 30  0000 C CNN
 	1    7550 5400
@@
 $EndComp
 $Comp
-L VCC #PWR025
+L VCC #PWR026
 U 1 1 4F4F36D4
 P 9750 5550
-F 0 "#PWR025" H 9750 5650 30  0001 C CNN
+F 0 "#PWR026" H 9750 5650 30  0001 C CNN
 F 1 "VCC" H 9750 5650 30  0000 C CNN
 	1    9750 5550
@@
 $EndComp
 $Comp
-L GND #PWR026
+L GND #PWR027
 U 1 1 4F4F36B2
 P 1500 5700
-F 0 "#PWR026" H 1500 5700 30  0001 C CNN
+F 0 "#PWR027" H 1500 5700 30  0001 C CNN
 F 1 "GND" H 1500 5630 30  0001 C CNN
 	1    1500 5700
@@
 $EndComp
 $Comp
-L +5V #PWR027
+L +5V #PWR028
 U 1 1 4F4F36A7
 P 1750 5300
-F 0 "#PWR027" H 1750 5390 20  0001 C CNN
+F 0 "#PWR028" H 1750 5390 20  0001 C CNN
 F 1 "+5V" H 1750 5390 30  0000 C CNN
 	1    1750 5300

Commit message: configured max1811 pin connections again
Connections:
- net +5V: no longer U1.1 (SELV)
- net GND: now also U1.1 (SELV)
