File: Controller_Version_2_single_PCB_attempt/Controller_Version_2_single_PCB_attempt.sch (KiCad schematic (older format))
At the start: 30 parts, among them IC1 ATTINY24-SS, J1 BATT, J2 NRF_conn, U1 MAX1811, U2 MAX1595, X1 USB-MB-S, X2 8MHz

Commit message: thougt i was ready, had fucked something up.. it should be okay now.
Parts:
- removed Ain1, N64, dw1: CONN_1, symbol CONN_1
- removed Batt1: CONN_3, symbol CONN_3
- removed Center_VCC1, Side_VCC1, Side_VCC2: CONN_2, symbol CONN_2
- added K?: CONN_3, symbol CONN_3
- added SW1: SW_PUSH, symbol SW_PUSH
Connections:
- net labels added: N64Serial, V_Batt_switched, Vchrg
- net labels removed: VCC
- wire segments 118 -> 129
Other:
- note added: "Battery Voltage Divider for the ADC"
- note added: "For feeding and interfacing the N64:"
- note added: "Is the ^SHDN net neccesary?"
- note removed: "Avoid routing errors, when on multiple boards:"
- note removed: "Battery Voltage Divider"
- note removed: "Below: Left PCB"
- note removed: "For feeding the N64:"
- note removed: "For feeding the center PCB:"
- note removed: "Top: 3.3V = Bottom VCC"
- note removed: "Top: Center PCB"
- note removed: "pin2 = Aout1"
- moved on the sheet: C1, C2, J1, X2

Commit message: All components are now fitted on the center PCB.. Routing this is going to be a challenge
Parts:
- gave numbers to parts that had none: 1

Commit message: almost done
Connections:
- net DGND is gone; now on net GND: C3.2, C4.2
- net Vchrg: now also R2.1
Changed lines of the file:
@@
-EESchema Schematic File Version 2  date 07-08-2012 10:05:19
+EESchema Schematic File Version 2  date 10-08-2012 17:50:50
 LIBS:power
 LIBS:device
@@
 Sheet 1 1
 Title ""
-Date "7 aug 2012"
+Date "10 aug 2012"
 Rev ""
 Comp ""
@@
 Comment4 ""
 $EndDescr
+Text GLabel 6450 1000 0    60   Input ~ 0
+Vchrg
+$Comp
+L GND #PWR01
+U 1 1 50252716
+P 2600 3650
+F 0 "#PWR01" H 2600 3650 30  0001 C CNN
+F 1 "GND" H 2600 3580 30  0001 C CNN
+	1    2600 3650
+	1    0    0    -1
+$EndComp
 Text Notes 6550 5150 0    60   ~ 0
 Is the ^SHDN net neccesary?
@@
 V_Batt_switched
 Wire Wire Line
-	5700 6450 5700 6700
+	5700 6450 5700 6600
+Wire Wire Line
+	5700 6600 5700 6700
 Connection ~ 6550 6700
 Wire Wire Line
-	6550 6450 6550 6700
+	6550 6700 6550 6450
 Wire Wire Line
 	6550 6450 6600 6450
 Wire Wire Line
-	6500 6700 6650 6700
+	6500 6700 6550 6700
+Wire Wire Line
+	6550 6700 6650 6700
 Wire Wire Line
 	4350 4250 4350 4200
@@
 Connection ~ 6100 2350
 Wire Wire Line
-	6100 2450 6100 1550
+	6100 2450 6100 2350
+Wire Wire Line
+	6100 2350 6100 1550
 Wire Wire Line
 	4650 1700 4550 1700
 Wire Wire Line
-	7800 5650 8100 5650
+	7800 5650 7850 5650
+Wire Wire Line
+	7850 5650 8100 5650
 Connection ~ 7200 5650
 Wire Wire Line
-	7050 5650 7300 5650
-Wire Wire Line
-	7200 5650 7200 5850
+	7050 5650 7200 5650
+Wire Wire Line
+	7200 5650 7300 5650
+Wire Wire Line
+	7200 5650 7200 5750
+Wire Wire Line
+	7200 5750 7200 5850
 Wire Wire Line
 	7400 6500 7400 6350
@@
 	8000 5550 8100 5550
 Wire Wire Line
-	9750 5150 9750 5550
+	9750 5150 9750 5250
+Wire Wire Line
+	9750 5250 9750 5550
 Wire Wire Line
 	6700 1000 6450 1000
@@
 	5200 2350 5200 2000
 Wire Wire Line
-	5550 2350 5200 2350
+	5200 2350 5450 2350
+Wire Wire Line
+	5450 2350 5550 2350
 Wire Wire Line
 	2550 6650 2550 6700
 Wire Wire Line
-	2550 7100 2550 6800
+	2550 7100 2550 7000
+Wire Wire Line
+	2550 7000 2550 6800
 Connection ~ 4450 7200
 Wire Wire Line
-	4450 7150 4450 7300
+	4450 7150 4450 7200
+Wire Wire Line
+	4450 7200 4450 7300
 Connection ~ 2600 3000
 Wire Wire Line
-	2800 3000 2350 3000
+	2800 3000 2600 3000
+Wire Wire Line
+	2600 3000 2350 3000
 Wire Wire Line
 	2800 3000 2800 3150
@@
 Connection ~ 2600 3550
 Wire Wire Line
-	2800 3550 2350 3550
+	2800 3550 2600 3550
+Wire Wire Line
+	2600 3550 2350 3550
 Wire Wire Line
 	1500 5700 1500 5350
@@
 	2150 5350 2700 5350
 Wire Wire Line
-	2150 6500 2700 6500
-Wire Wire Line
-	2150 6350 2150 6500
-Wire Wire Line
-	2150 5300 2150 5400
-Wire Wire Line
-	4450 6600 4450 6750
+	2700 6500 2150 6500
+Wire Wire Line
+	2150 6500 2150 6450
+Wire Wire Line
+	2150 6450 2150 6350
+Wire Wire Line
+	2150 5300 2150 5350
+Wire Wire Line
+	2150 5350 2150 5400
+Wire Wire Line
+	4450 6600 4450 6700
+Wire Wire Line
+	4450 6700 4450 6750
 Wire Wire Line
 	3900 7000 4000 7000
@@
 Connection ~ 5700 7000
 Wire Wire Line
-	5700 7150 5700 6900
+	5700 7150 5700 7000
+Wire Wire Line
+	5700 7000 5700 6900
 Wire Wire Line
 	5350 7000 5700 7000
@@
 	2600 2950 2600 3000
 Wire Wire Line
-	3900 6700 4800 6700
+	3900 6700 4450 6700
+Wire Wire Line
+	4450 6700 4800 6700
 Wire Wire Line
 	4800 6700 4800 6750
@@
 	4800 7200 4450 7200
 Wire Wire Line
-	5550 1550 5200 1550
+	5550 1550 5450 1550
+Wire Wire Line
+	5450 1550 5200 1550
 Wire Wire Line
 	5200 1550 5200 1900
@@
 	2350 1000 2450 1000
 Wire Wire Line
-	7200 1000 7400 1000
+	7200 1000 7300 1000
+Wire Wire Line
+	7300 1000 7400 1000
 Wire Wire Line
 	7900 1000 8000 1000
@@
 	9700 5850 9700 5950
 Wire Wire Line
-	9950 5550 9950 5850
-Wire Wire Line
-	9600 5550 9950 5550
+	9950 5850 9950 5550
+Wire Wire Line
+	9950 5550 9750 5550
+Wire Wire Line
+	9750 5550 9600 5550
 Connection ~ 9750 5550
 Wire Wire Line
@@
 	8050 5850 8050 5950
 Wire Wire Line
-	7200 6350 7200 6250
-Wire Wire Line
-	7600 6350 7600 6250
-Wire Wire Line
-	7200 6350 7600 6350
+	7200 6250 7200 6350
+Wire Wire Line
+	7600 6250 7600 6350
+Wire Wire Line
+	7600 6350 7400 6350
+Wire Wire Line
+	7400 6350 7200 6350
 Connection ~ 7400 6350
 Connection ~ 7200 5750
 Wire Wire Line
-	7200 5750 8100 5750
+	7200 5750 7600 5750
+Wire Wire Line
+	7600 5750 8100 5750
 Wire Wire Line
 	2450 2200 2350 2200
 Wire Wire Line
 	2350 2200 2350 2300
-Wire Wire Line
-	6450 1000 6450 850
 Wire Wire Line
 	5200 2000 4550 2000
@@
 $EndComp
 $Comp
-L +BATT #PWR01
-U 1 1 50190B42
-P 6450 900
-F 0 "#PWR01" H 6450 850 20  0001 C CNN
-F 1 "+BATT" H 6450 1000 30  0000 C CNN
-	1    6450 900
-	1    0    0    -1
-$EndComp
-$Comp
-L +3.3V #PWR02
+L +3.3V #PWR03
 U 1 1 501904C7
 P 9750 5150
-F 0 "#PWR02" H 9750 5110 30  0001 C CNN
+F 0 "#PWR03" H 9750 5110 30  0001 C CNN
 F 1 "+3.3V" H 9750 5260 30  0000 C CNN
 	1    9750 5150
@@
 $EndComp
 $Comp
-L GND #PWR03
+L GND #PWR04
 U 1 1 50190402
 P 8000 1100
-F 0 "#PWR03" H 8000 1100 30  0001 C CNN
+F 0 "#PWR04" H 8000 1100 30  0001 C CNN
 F 1 "GND" H 8000 1030 30  0001 C CNN
 	1    8000 1100
@@
 $EndComp
 $Comp
-L GND #PWR04
+L GND #PWR05
 U 1 1 501903FD
 P 6750 2700
-F 0 "#PWR04" H 6750 2700 30  0001 C CNN
+F 0 "#PWR05" H 6750 2700 30  0001 C CNN
 F 1 "GND" H 6750 2630 30  0001 C CNN
 	1    6750 2700
@@
 $EndComp
 $Comp
-L GND #PWR05
+L GND #PWR06
 U 1 1 501903F3
 P 6100 2450
-F 0 "#PWR05" H 6100 2450 30  0001 C CNN
+F 0 "#PWR06" H 6100 2450 30  0001 C CNN
 F 1 "GND" H 6100 2380 30  0001 C CNN
 	1    6100 2450
@@
 $EndComp
 $Comp
-L GND #PWR06
+L GND #PWR07
 U 1 1 501903E5
 P 2350 2300
-F 0 "#PWR06" H 2350 2300 30  0001 C CNN
+F 0 "#PWR07" H 2350 2300 30  0001 C CNN
 F 1 "GND" H 2350 2230 30  0001 C CNN
 	1    2350 2300
@@
 $EndComp
 $Comp
-L GND #PWR07
+L GND #PWR08
 U 1 1 4FEA19AE
 P 8050 5950
-F 0 "#PWR07" H 8050 5950 30  0001 C CNN
+F 0 "#PWR08" H 8050 5950 30  0001 C CNN
 F 1 "GND" H 8050 5880 30  0001 C CNN
 	1    8050 5950
@@
 approx 3mA@8MHz@3v3
 $Comp
-L +3.3V #PWR08
+L +3.3V #PWR09
 U 1 1 4FE6ECED
 P 2350 1000
-F 0 "#PWR08" H 2350 960 30  0001 C CNN
+F 0 "#PWR09" H 2350 960 30  0001 C CNN
 F 1 "+3.3V" H 2350 1110 30  0000 C CNN
 	1    2350 1000
@@
 $EndComp
 $Comp
-L +5V #PWR09
+L +5V #PWR010
 U 1 1 4FE08C10
 P 2550 6650
-F 0 "#PWR09" H 2550 6740 20  0001 C CNN
+F 0 "#PWR010" H 2550 6740 20  0001 C CNN
 F 1 "+5V" H 2550 6740 30  0000 C CNN
 	1    2550 6650
@@
 $EndComp
 $Comp
-L +3.3V #PWR010
+L +3.3V #PWR011
 U 1 1 4FC72ABF
 P 8300 2300
-F 0 "#PWR010" H 8300 2260 30  0001 C CNN
+F 0 "#PWR011" H 8300 2260 30  0001 C CNN
 F 1 "+3.3V" H 8300 2410 30  0000 C CNN
 	1    8300 2300
@@
 $EndComp
 $Comp
-L +3.3V #PWR011
+L +3.3V #PWR012
 U 1 1 4FC72AB1
 P 2600 2950
-F 0 "#PWR011" H 2600 2910 30  0001 C CNN
+F 0 "#PWR012" H 2600 2910 30  0001 C CNN
 F 1 "+3.3V" H 2600 3060 30  0000 C CNN
 	1    2600 2950
@@
 $EndComp
 $Comp
-L +3.3V #PWR012
+L +3.3V #PWR013
 U 1 1 4FC72AA1
 P 4350 3950
-F 0 "#PWR012" H 4350 3910 30  0001 C CNN
+F 0 "#PWR013" H 4350 3910 30  0001 C CNN
 F 1 "+3.3V" H 4350 4060 30  0000 C CNN
 	1    4350 3950
@@
 $EndComp
 $Comp
-L GND #PWR013
+L GND #PWR014
 U 1 1 4FC72A57
 P 4350 4250
-F 0 "#PWR013" H 4350 4250 30  0001 C CNN
+F 0 "#PWR014" H 4350 4250 30  0001 C CNN
 F 1 "GND" H 4350 4180 30  0001 C CNN
 	1    4350 4250
 	1    0    0    -1
 $EndComp
-$Comp
-L DGND #PWR014
-U 1 1 4FC72A04
-P 2600 3650
-F 0 "#PWR014" H 2600 3650 40  0001 C CNN
-F 1 "DGND" H 2600 3580 40  0000 C CNN
-	1    2600 3650
-	1    0    0    -1
-$EndComp

Commit message: got a new idea..
Changed lines of the file:
@@
-EESchema Schematic File Version 2  date 10-08-2012 17:50:50
+EESchema Schematic File Version 2  date 10-08-2012 18:13:49
 LIBS:power
 LIBS:device
@@
 V_Batt_switched
 Wire Wire Line
-	5700 6450 5700 6600
-Wire Wire Line
-	5700 6600 5700 6700
+	5700 6450 5700 6700
 Connection ~ 6550 6700
 Wire Wire Line
-	6550 6700 6550 6450
+	6550 6450 6550 6700
 Wire Wire Line
 	6550 6450 6600 6450
 Wire Wire Line
-	6500 6700 6550 6700
-Wire Wire Line
-	6550 6700 6650 6700
+	6500 6700 6650 6700
 Wire Wire Line
 	4350 4250 4350 4200
@@
 Connection ~ 6100 2350
 Wire Wire Line
-	6100 2450 6100 2350
-Wire Wire Line
-	6100 2350 6100 1550
+	6100 2450 6100 1550
 Wire Wire Line
 	4650 1700 4550 1700
 Wire Wire Line
-	7800 5650 7850 5650
-Wire Wire Line
-	7850 5650 8100 5650
+	7800 5650 8100 5650
 Connection ~ 7200 5650
 Wire Wire Line
-	7050 5650 7200 5650
-Wire Wire Line
-	7200 5650 7300 5650
-Wire Wire Line
-	7200 5650 7200 5750
-Wire Wire Line
-	7200 5750 7200 5850
+	7050 5650 7300 5650
+Wire Wire Line
+	7200 5650 7200 5850
 Wire Wire Line
 	7400 6500 7400 6350
@@
 	8000 5550 8100 5550
 Wire Wire Line
-	9750 5150 9750 5250
-Wire Wire Line
-	9750 5250 9750 5550
+	9750 5150 9750 5550
 Wire Wire Line
 	6700 1000 6450 1000
@@
 	5200 2350 5200 2000
 Wire Wire Line
-	5200 2350 5450 2350
-Wire Wire Line
-	5450 2350 5550 2350
+	5550 2350 5200 2350
 Wire Wire Line
 	2550 6650 2550 6700
 Wire Wire Line
-	2550 7100 2550 7000
-Wire Wire Line
-	2550 7000 2550 6800
+	2550 7100 2550 6800
 Connection ~ 4450 7200
 Wire Wire Line
-	4450 7150 4450 7200
-Wire Wire Line
-	4450 7200 4450 7300
+	4450 7150 4450 7300
 Connection ~ 2600 3000
 Wire Wire Line
-	2800 3000 2600 3000
-Wire Wire Line
-	2600 3000 2350 3000
+	2800 3000 2350 3000
 Wire Wire Line
 	2800 3000 2800 3150
@@
 Connection ~ 2600 3550
 Wire Wire Line
-	2800 3550 2600 3550
-Wire Wire Line
-	2600 3550 2350 3550
+	2800 3550 2350 3550
 Wire Wire Line
 	1500 5700 1500 5350
@@
 	2150 5350 2700 5350
 Wire Wire Line
-	2700 6500 2150 6500
-Wire Wire Line
-	2150 6500 2150 6450
-Wire Wire Line
-	2150 6450 2150 6350
-Wire Wire Line
-	2150 5300 2150 5350
-Wire Wire Line
-	2150 5350 2150 5400
-Wire Wire Line
-	4450 6600 4450 6700
-Wire Wire Line
-	4450 6700 4450 6750
+	2150 6500 2700 6500
+Wire Wire Line
+	2150 6350 2150 6500
+Wire Wire Line
+	2150 5300 2150 5400
+Wire Wire Line
+	4450 6600 4450 6750
 Wire Wire Line
 	3900 7000 4000 7000
@@
 Connection ~ 5700 7000
 Wire Wire Line
-	5700 7150 5700 7000
-Wire Wire Line
-	5700 7000 5700 6900
+	5700 7150 5700 6900
 Wire Wire Line
 	5350 7000 5700 7000
@@
 	2600 2950 2600 3000
 Wire Wire Line
-	3900 6700 4450 6700
-Wire Wire Line
-	4450 6700 4800 6700
+	3900 6700 4800 6700
 Wire Wire Line
 	4800 6700 4800 6750
@@
 	4800 7200 4450 7200
 Wire Wire Line
-	5550 1550 5450 1550
-Wire Wire Line
-	5450 1550 5200 1550
+	5550 1550 5200 1550
 Wire Wire Line
 	5200 1550 5200 1900
@@
 	2350 1000 2450 1000
 Wire Wire Line
-	7200 1000 7300 1000
-Wire Wire Line
-	7300 1000 7400 1000
+	7200 1000 7400 1000
 Wire Wire Line
 	7900 1000 8000 1000
@@
 	9700 5850 9700 5950
 Wire Wire Line
-	9950 5850 9950 5550
-Wire Wire Line
-	9950 5550 9750 5550
-Wire Wire Line
-	9750 5550 9600 5550
+	9950 5550 9950 5850
+Wire Wire Line
+	9600 5550 9950 5550
 Connection ~ 9750 5550
 Wire Wire Line
@@
 	8050 5850 8050 5950
 Wire Wire Line
-	7200 6250 7200 6350
-Wire Wire Line
-	7600 6250 7600 6350
-Wire Wire Line
-	7600 6350 7400 6350
-Wire Wire Line
-	7400 6350 7200 6350
+	7200 6350 7200 6250
+Wire Wire Line
+	7600 6350 7600 6250
+Wire Wire Line
+	7200 6350 7600 6350
 Connection ~ 7400 6350
 Connection ~ 7200 5750
 Wire Wire Line
-	7200 5750 7600 5750
-Wire Wire Line
-	7600 5750 8100 5750
+	7200 5750 8100 5750
 Wire Wire Line
 	2450 2200 2350 2200
@@
 $EndComp
 $Comp
-L +3.3V #PWR03
+L +3.3V #PWR02
 U 1 1 501904C7
 P 9750 5150
-F 0 "#PWR03" H 9750 5110 30  0001 C CNN
+F 0 "#PWR02" H 9750 5110 30  0001 C CNN
 F 1 "+3.3V" H 9750 5260 30  0000 C CNN
 	1    9750 5150
@@
 $EndComp
 $Comp
-L GND #PWR04
+L GND #PWR03
 U 1 1 50190402
 P 8000 1100
-F 0 "#PWR04" H 8000 1100 30  0001 C CNN
+F 0 "#PWR03" H 8000 1100 30  0001 C CNN
 F 1 "GND" H 8000 1030 30  0001 C CNN
 	1    8000 1100
@@
 $EndComp
 $Comp
-L GND #PWR05
+L GND #PWR04
 U 1 1 501903FD
 P 6750 2700
-F 0 "#PWR05" H 6750 2700 30  0001 C CNN
+F 0 "#PWR04" H 6750 2700 30  0001 C CNN
 F 1 "GND" H 6750 2630 30  0001 C CNN
 	1    6750 2700
@@
 $EndComp
 $Comp
-L GND #PWR06
+L GND #PWR05
 U 1 1 501903F3
 P 6100 2450
-F 0 "#PWR06" H 6100 2450 30  0001 C CNN
+F 0 "#PWR05" H 6100 2450 30  0001 C CNN
 F 1 "GND" H 6100 2380 30  0001 C CNN
 	1    6100 2450
@@
 $EndComp
 $Comp
-L GND #PWR07
+L GND #PWR06
 U 1 1 501903E5
 P 2350 2300
-F 0 "#PWR07" H 2350 2300 30  0001 C CNN
+F 0 "#PWR06" H 2350 2300 30  0001 C CNN
 F 1 "GND" H 2350 2230 30  0001 C CNN
 	1    2350 2300
@@
 $EndComp
 $Comp
-L GND #PWR08
+L GND #PWR07
 U 1 1 4FEA19AE
 P 8050 5950
-F 0 "#PWR08" H 8050 5950 30  0001 C CNN
+F 0 "#PWR07" H 8050 5950 30  0001 C CNN
 F 1 "GND" H 8050 5880 30  0001 C CNN
 	1    8050 5950
@@
 approx 3mA@8MHz@3v3
 $Comp
-L +3.3V #PWR09
+L +3.3V #PWR08
 U 1 1 4FE6ECED
 P 2350 1000
-F 0 "#PWR09" H 2350 960 30  0001 C CNN
+F 0 "#PWR08" H 2350 960 30  0001 C CNN
 F 1 "+3.3V" H 2350 1110 30  0000 C CNN
 	1    2350 1000
@@
 $EndComp
 $Comp
-L +5V #PWR010
+L +5V #PWR09
 U 1 1 4FE08C10
 P 2550 6650
-F 0 "#PWR010" H 2550 6740 20  0001 C CNN
+F 0 "#PWR09" H 2550 6740 20  0001 C CNN
 F 1 "+5V" H 2550 6740 30  0000 C CNN
 	1    2550 6650
@@
 $EndComp
 $Comp
-L +3.3V #PWR011
+L +3.3V #PWR010
 U 1 1 4FC72ABF
 P 8300 2300
-F 0 "#PWR011" H 8300 2260 30  0001 C CNN
+F 0 "#PWR010" H 8300 2260 30  0001 C CNN
 F 1 "+3.3V" H 8300 2410 30  0000 C CNN
 	1    8300 2300
@@
 $EndComp
 $Comp
-L +3.3V #PWR012
+L +3.3V #PWR011
 U 1 1 4FC72AB1
 P 2600 2950
-F 0 "#PWR012" H 2600 2910 30  0001 C CNN
+F 0 "#PWR011" H 2600 2910 30  0001 C CNN
 F 1 "+3.3V" H 2600 3060 30  0000 C CNN
 	1    2600 2950
@@
 $EndComp
 $Comp
-L +3.3V #PWR013
+L +3.3V #PWR012
 U 1 1 4FC72AA1
 P 4350 3950
-F 0 "#PWR013" H 4350 3910 30  0001 C CNN
+F 0 "#PWR012" H 4350 3910 30  0001 C CNN
 F 1 "+3.3V" H 4350 4060 30  0000 C CNN
 	1    4350 3950
@@
 $EndComp
 $Comp
-L GND #PWR014
+L GND #PWR013
 U 1 1 4FC72A57
 P 4350 4250
-F 0 "#PWR014" H 4350 4250 30  0001 C CNN
+F 0 "#PWR013" H 4350 4250 30  0001 C CNN
 F 1 "GND" H 4350 4180 30  0001 C CNN
 	1    4350 4250
@@
 CE
 $Comp
-L GND #PWR015
+L GND #PWR014
 U 1 1 4F5F6BBA
 P 7400 6500
-F 0 "#PWR015" H 7400 6500 30  0001 C CNN
+F 0 "#PWR014" H 7400 6500 30  0001 C CNN
 F 1 "GND" H 7400 6430 30  0001 C CNN
 	1    7400 6500
@@
 $EndComp
 $Comp
-L GND #PWR016
+L GND #PWR015
 U 1 1 4F5F6A53
 P 9950 6500
-F 0 "#PWR016" H 9950 6500 30  0001 C CNN
+F 0 "#PWR015" H 9950 6500 30  0001 C CNN
 F 1 "GND" H 9950 6430 30  0001 C CNN
 	1    9950 6500
@@
 $EndComp
 $Comp
-L GND #PWR017
+L GND #PWR016
 U 1 1 4F5F6856
 P 9700 5950
-F 0 "#PWR017" H 9700 5950 30  0001 C CNN
+F 0 "#PWR016" H 9700 5950 30  0001 C CNN
 F 1 "GND" H 9700 5880 30  0001 C CNN
 	1    9700 5950
@@
 $EndComp
 $Comp
-L +5V #PWR018
+L +5V #PWR017
 U 1 1 4F4F395E
 P 2150 5300
-F 0 "#PWR018" H 2150 5390 20  0001 C CNN
+F 0 "#PWR017" H 2150 5390 20  0001 C CNN
 F 1 "+5V" H 2150 5390 30  0000 C CNN
 	1    2150 5300
@@
 $EndComp
 $Comp
-L +5V #PWR019
+L +5V #PWR018
 U 1 1 4F4F393F
 P 4450 6600
-F 0 "#PWR019" H 4450 6690 20  0001 C CNN
+F 0 "#PWR018" H 4450 6690 20  0001 C CNN
 F 1 "+5V" H 4450 6690 30  0000 C CNN
 	1    4450 6600
@@
 $EndComp
 $Comp
-L GND #PWR020
+L GND #PWR019
 U 1 1 4F4F3934
 P 4450 7300
-F 0 "#PWR020" H 4450 7300 30  0001 C CNN
+F 0 "#PWR019" H 4450 7300 30  0001 C CNN
 F 1 "GND" H 4450 7230 30  0001 C CNN
 	1    4450 7300
@@
 $EndComp
 $Comp
-L GND #PWR021
+L GND #PWR020
 U 1 1 4F4F38CA
 P 4000 7100
-F 0 "#PWR021" H 4000 7100 30  0001 C CNN
+F 0 "#PWR020" H 4000 7100 30  0001 C CNN
 F 1 "GND" H 4000 7030 30  0001 C CNN
 	1    4000 7100
@@
 $EndComp
 $Comp
-L GND #PWR022
+L GND #PWR021
 U 1 1 4F4F38C1
 P 2550 7100
-F 0 "#PWR022" H 2550 7100 30  0001 C CNN
+F 0 "#PWR021" H 2550 7100 30  0001 C CNN
 F 1 "GND" H 2550 7030 30  0001 C CNN
 	1    2550 7100
@@
 $EndComp
 $Comp
-L GND #PWR023
+L GND #PWR022
 U 1 1 4F4F372C
 P 5700 7150
-F 0 "#PWR023" H 5700 7150 30  0001 C CNN
+F 0 "#PWR022" H 5700 7150 30  0001 C CNN
 F 1 "GND" H 5700 7080 30  0001 C CNN
 	1    5700 7150
@@
 $EndComp
 $Comp
-L GND #PWR024
+L GND #PWR023
 U 1 1 4F4F36B2
 P 1500 5700
-F 0 "#PWR024" H 1500 5700 30  0001 C CNN
+F 0 "#PWR023" H 1500 5700 30  0001 C CNN
 F 1 "GND" H 1500 5630 30  0001 C CNN
 	1    1500 5700
@@
 $EndComp
 $Comp
-L +5V #PWR025
+L +5V #PWR024
 U 1 1 4F4F36A7
 P 1750 5300
-F 0 "#PWR025" H 1750 5390 20  0001 C CNN
+F 0 "#PWR024" H 1750 5390 20  0001 C CNN
 F 1 "+5V" H 1750 5390 30  0000 C CNN
 	1    1750 5300
